File: N-V1-R2/petkn.sch (KiCad schematic (older format))
At the start: 88 parts, among them J1 Conn_01x20, J2 Conn_02x03_Odd_Even, J3 LINK3, J4 Conn_01x20, J5 SPACE1, J6 SPACE2, J67 LINK67, SW1 KP \"=\", SW10 KP \"0\", SW11 R SHIFT, SW12 \">\", SW13 NC, SW14 \"]\", SW15 \"@\", SW16 L SHIFT, SW17 KP \"+\", SW18 KP \"2\", SW19 NC, SW2 KP \".\", SW20 \"?\", SW21 \",\", SW22 \"N\", SW23 \"V\", SW24 \"X\", SW25 KP \"3\", SW26 KP \"1\", SW27 RETURN, SW28 \";\", SW29 \"M\", SW3 NC ($10), SW30 \"B\", SW31 \"C\", SW32 \"Z\", SW320 S LOCK, SW33 KP \"*\", SW34 KP \"5\", SW35 NC, SW36 \":\", SW37 \"K\", SW38 \"H\", SW39 \"F\", SW4 STOP, SW40 \"S\", SW41 KP \"6\", SW42 KP \"4\", SW43 NC, SW44 \"L\", SW45 \"J\", SW46 \"G\", SW47 \"D\", SW48 \"A\", SW49 KP \"/\", SW5 \"<\", SW50 KP \"8\", SW51 NC, SW52 \"P\", SW53 \"I\", SW54 \"Y\", SW55 \"R\", SW56 \"W\", SW57 KP \"9\", SW58 KP \"7\", SW59 U ARROW, SW6 SPACE, SW60 \"O\", SW61 \"U\", SW62 \"T\", SW63 \"E\", SW64 \"Q\", SW65 INS/DEL, SW66 UP/DOWN, SW67 NC ($0A), SW68 \")\", SW69 \"\\\", SW7 \"[\", SW70 \"'\", SW71 \"$\", SW72 QUOTE, SW73 LEFT/RIGHT, SW74 CLR/HOME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

Commit message: Update N-V1-R2 schematic
Updated schematic to remove unused switches, and replace with some more
descriptive text to make alternate configurations clearer/
Parts:
- removed SW13, SW19, SW35, SW43, SW51: NC, Button_Switch_Keyboard:SW_Cherry_MX_1.00u_PCB, symbol Switch:SW_Push
Connections:
- wire segments 238 -> 233
Other:
- note added: "<- SHIFT-LOCK\n\n<- ALT (SW51)"
- note added: "C8 C7 C6 C5 C4 C3 C2 C1"
- note added: "LOCK"
- note added: "Locking MX switches are hard to get, but if you have\none it can be used, or it can be jumpered for SW51.\n"
- note added: "N/C\n$0A"
- note added: "N/C\n$10"
- note added: "N/C\nALT"
- note added: "R1 R2 R3 R4 R5 R6 R7 R8 R9 R10"
- note added: "SHIFT-LOCK / SWITCH51"
- note removed: "<- SHIFT-LOCK\n\n<- ALT"
- note removed: "Locking MX switches are hard to get,\nbut If you have one it can be used.\n"
- note removed: "SHIFT-LOCK"
Changed lines of the file:
@@
 	3650 1175 3650 1575
 Connection ~ 3650 1575
-Wire Wire Line
-	3650 1575 3650 2100
 $Comp
 L Switch:SW_Push SW6
@@
 Wire Wire Line
 	3550 2100 3550 2275
-$Comp
-L Switch:SW_Push SW13
-U 1 1 5EE76D8A
-P 3850 2100
-F 0 "SW13" H 3850 2385 50  0000 C CNN
-F 1 "NC" H 3850 2294 50  0000 C CNN
-F 2 "Button_Switch_Keyboard:SW_Cherry_MX_1.00u_PCB" H 3850 2300 50  0001 C CNN
-F 3 "~" H 3850 2300 50  0001 C CNN
-	1    3850 2100
-	1    0    0    -1
-$EndComp
 Wire Wire Line
 	4050 2100 4050 2275
@@
 	2125 2100 2125 2625
 Connection ~ 2650 2100
-Wire Wire Line
-	2650 2100 2650 2625
 Connection ~ 3150 2100
 Wire Wire Line
 	3150 2100 3150 2625
-Connection ~ 3650 2100
-Wire Wire Line
-	3650 2100 3650 2625
 Connection ~ 4150 2100
 Wire Wire Line
@@
 	1    0    0    -1
 $EndComp
-$Comp
-L Switch:SW_Push SW19
-U 1 1 5EE7FE66
-P 2850 2625
-F 0 "SW19" H 2850 2910 50  0000 C CNN
-F 1 "NC" H 2850 2819 50  0000 C CNN
-F 2 "Button_Switch_Keyboard:SW_Cherry_MX_1.00u_PCB" H 2850 2825 50  0001 C CNN
-F 3 "~" H 2850 2825 50  0001 C CNN
-	1    2850 2625
-	1    0    0    -1
-$EndComp
 Wire Wire Line
 	3050 2625 3050 2800
@@
 Wire Wire Line
 	2125 2625 2125 3150
-Connection ~ 2650 2625
-Wire Wire Line
-	2650 2625 2650 3150
 Connection ~ 3150 2625
 Wire Wire Line
@@
 	3150 3150 3150 3675
 Wire Wire Line
-	2650 3150 2650 3675
-Wire Wire Line
 	2125 3150 2125 3675
 Wire Wire Line
@@
 	1    0    0    -1
 $EndComp
-$Comp
-L Switch:SW_Push SW35
-U 1 1 5EEF89EB
-P 2850 3675
-F 0 "SW35" H 2850 3960 50  0000 C CNN
-F 1 "NC" H 2850 3869 50  0000 C CNN
-F 2 "Button_Switch_Keyboard:SW_Cherry_MX_1.00u_PCB" H 2850 3875 50  0001 C CNN
-F 3 "~" H 2850 3875 50  0001 C CNN
-	1    2850 3675
-	1    0    0    -1
-$EndComp
 Wire Wire Line
 	3050 3675 3050 3850
@@
 Wire Wire Line
 	2125 3675 2125 4200
-Connection ~ 2650 3675
-Wire Wire Line
-	2650 3675 2650 4200
 Connection ~ 3150 3675
 Wire Wire Line
@@
 	1    0    0    -1
 $EndComp
-$Comp
-L Switch:SW_Push SW43
-U 1 1 5EF1D9B0
-P 2850 4200
-F 0 "SW43" H 2850 4485 50  0000 C CNN
-F 1 "NC" H 2850 4394 50  0000 C CNN
-F 2 "Button_Switch_Keyboard:SW_Cherry_MX_1.00u_PCB" H 2850 4400 50  0001 C CNN
-F 3 "~" H 2850 4400 50  0001 C CNN
-	1    2850 4200
-	1    0    0    -1
-$EndComp
 Wire Wire Line
 	3050 4200 3050 4375
@@
 	1    0    0    -1
 $EndComp
-$Comp
-L Switch:SW_Push SW51
-U 1 1 5EF3BE66
-P 2850 4725
-F 0 "SW51" H 2850 5010 50  0000 C CNN
-F 1 "NC" H 2850 4919 50  0000 C CNN
-F 2 "Button_Switch_Keyboard:SW_Cherry_MX_1.00u_PCB" H 2850 4925 50  0001 C CNN
-F 3 "~" H 2850 4925 50  0001 C CNN
-	1    2850 4725
-	1    0    0    -1
-$EndComp
 Wire Wire Line
 	3050 4725 3050 4900
@@
 Wire Wire Line
 	3150 4200 3150 4725
-Connection ~ 2650 4200
-Wire Wire Line
-	2650 4200 2650 4725
 Connection ~ 2125 4200
 Wire Wire Line
@@
 Wire Wire Line
 	2125 4725 2125 5250
-Connection ~ 2650 4725
-Wire Wire Line
-	2650 4725 2650 5250
 Connection ~ 3150 4725
 Wire Wire Line
@@
 Text Notes 9850 1100 0    61   ~ 0
 GROUND
-Text Notes 1025 6675 0    79   ~ 0
+Text Notes 1025 6900 0    79   ~ 0
 KP = Keypad. SW numbers correspond to position in matrix. R/C match connector.
 Text Notes 8750 7100 0    118  ~ 24
@@
 Text Notes 9425 925  0    118  ~ 24
 CONNECTORS
-Text Notes 575  7175 0    118  ~ 24
+Text Notes 575  7275 0    118  ~ 24
 PET/CBM "N" KEYBOARD
-Text Notes 600  7625 0    61   ~ 0
+Text Notes 600  7725 0    61   ~ 0
 Standard "N" layout with the following changes:\n- SPACEBAR now 6.25U. Two keys added beside it.\n- SHIFTLOCK is configurable\n- Jumpers to make extra keys work as SPACEBAR or Alternate\n
 Text Notes 8700 6425 0    118  ~ 0
@@
 R10
 Text Notes 6200 1275 0    87   ~ 17
-SHIFT-LOCK
+SHIFT-LOCK / SWITCH51
 Text Notes 6200 1475 0    61   ~ 0
-Locking MX switches are hard to get,\nbut If you have one it can be used.\n
+Locking MX switches are hard to get, but if you have\none it can be used, or it can be jumpered for SW51.\n
 Text Notes 8125 1925 0    61   ~ 0
-<- SHIFT-LOCK\n\n<- ALT
+<- SHIFT-LOCK\n\n<- ALT (SW51)
 $Comp
 L Connector_Generic:Conn_01x20 J4
@@
 Text GLabel 6825 4100 2    50   Input ~ 0
 XR67
-Text Notes 3725 7350 0    79   ~ 16
+Text Notes 3725 7450 0    79   ~ 16
 RELEASES:\n* N-V1-R1 PCB Submitted 2020-12-18\n* N-V1-R2 PCB Updated 2021-03-31
 Text Notes 6225 4625 0    87   ~ 17
@@
 	1    0    0    -1
 $EndComp
+Text Notes 1625 6750 0    189  ~ 38
+C8 C7 C6 C5 C4 C3 C2 C1
+Text Notes 5900 6450 1    193  ~ 39
+R1 R2 R3 R4 R5 R6 R7 R8 R9 R10
+Text Notes 2725 1625 0    87   ~ 17
+N/C\n$10
+Text Notes 2725 5775 0    87   ~ 17
+N/C\n$0A
+Wire Wire Line
+	2650 2100 2650 3150
+Wire Wire Line
+	2650 3150 2650 5250
+Wire Wire Line
+	3650 1575 3650 2625
+Text Notes 5200 2250 0    87   ~ 17
+LOCK
+Text Notes 2725 4775 0    87   ~ 17
+N/C\nALT
 $EndSCHEMATC
